Commit message: Updated urdf

File: iai_tiago_description/urdf/tiago_from_our_robot.urdf (robot description, URDF)
Before this commit: robot tiago_dual, 84 links, 83 joints
Links:
- link arm_left_1_link: geometry collision mesh filename=package://tiago_description/meshes/arm/arm_1_collision.stl scale=1 -1 -1; visual mesh filename=package://tiago_description/meshes/arm/arm_1.stl scale=1 -1 -1
- link arm_left_2_link: geometry collision mesh filename=package://tiago_description/meshes/arm/arm_2_collision.stl scale=1 1 -1; visual mesh filename=package://tiago_description/meshes/arm/arm_2.stl scale=1 1 -1
- link arm_left_3_link: geometry collision mesh filename=package://tiago_description/meshes/arm/arm_3_collision.stl scale=1 1 -1; visual mesh filename=package://tiago_description/meshes/arm/arm_3.stl scale=1 1 -1
- link arm_left_4_link: geometry collision mesh filename=package://tiago_description/meshes/arm/arm_4_collision.stl scale=-1 -1 -1; visual mesh filename=package://tiago_description/meshes/arm/arm_4.stl scale=-1 -1 -1
- link arm_right_1_link: geometry collision mesh filename=package://tiago_description/meshes/arm/arm_1_collision.stl scale=1 -1 1; visual mesh filename=package://tiago_description/meshes/arm/arm_1.stl scale=1 -1 1
- link arm_right_2_link: geometry collision mesh filename=package://tiago_description/meshes/arm/arm_2_collision.stl scale=1 1 1; visual mesh filename=package://tiago_description/meshes/arm/arm_2.stl scale=1 1 1
- link arm_right_3_link: geometry collision mesh filename=package://tiago_description/meshes/arm/arm_3_collision.stl scale=1 1 1; visual mesh filename=package://tiago_description/meshes/arm/arm_3.stl scale=1 1 1
- link arm_right_4_link: geometry collision mesh filename=package://tiago_description/meshes/arm/arm_4_collision.stl scale=1 1 1; visual mesh filename=package://tiago_description/meshes/arm/arm_4.stl scale=1 1 1
